Commit message: panda now has mount_point instead of world as urdf base link

File: franka_bringup/srdf/panda.srdf_macro.xacro (robot description, xacro)
@@ -5,5 +5,5 @@
       <chain base_link="${tf_prefix}base_link" tip_link="${tf_prefix}tool0" />
     </group>
-    <virtual_joint name="virtual_joint" type="fixed" parent_frame="world" child_link="${tf_prefix}base_link"/>
+    <virtual_joint name="virtual_joint" type="fixed" parent_frame="world" child_link="${tf_prefix}mount_point"/>
     <group_state name="home" group="${tf_prefix}manipulator">
       <joint name="${tf_prefix}joint_1" value="0"/>

File: franka_description/urdf/panda.urdf.xacro (robot description, xacro)
@@ -4,5 +4,4 @@
   <xacro:arg name="robot_ip" default=""/> <!-- IP address or hostname of the robot" -->
   <xacro:arg name="use_mock_hardware" default="false"/>
-  <link name="world" />
   <xacro:include filename="$(find franka_description)/urdf/panda.urdf_macro.xacro"/>
   <xacro:panda_urdf_macro tf_prefix="$(arg tf_prefix)" safety_distance="0.03"/>

File: franka_description/urdf/panda.urdf_macro.xacro (robot description, xacro)
@@ -4,7 +4,8 @@
   <!-- tf_prefix: Namespace of the panda arm. Serves to differentiate between arms in case of multiple instances. -->
   <xacro:macro name="panda_urdf_macro" params="tf_prefix safety_distance:=0">
+    <link name="${tf_prefix}mount_point"/>
     <joint name="${tf_prefix}base_joint" type="fixed">
       <origin xyz="0 0 0" rpy="0 0 0" />
-      <parent link="world" />
+      <parent link="${tf_prefix}mount_point" />
       <child link="${tf_prefix}base_link" />
     </joint>
